Commit message: Update ur5 urdf

File: description/ur5/urdf/ur5.urdf (robot description, URDF)
Before this commit: robot ur5, 13 links, 12 joints
Links:
- removed link wall
Joints:
- removed joint world_to_wall_joint

Commit message: FEAT: Add dynamics MPC self-collision constraints and visualization
- Add shared dynamics self-collision constraint/evaluator for ID and FD MPC
- Support per-position and per-velocity state limit activation
- Add self-collision hard-stop fallback into impedance hold
- Add policy self-collision distance visualization markers
- Reuse shared `ocs2.task.selfCollision` config for controllers and visualization
- Update UR5/dual-UR5 controller YAML and RViz marker display

File: description/ur5/urdf/ur5.urdf (robot description, URDF)
Before this commit: robot ur5, 12 links, 11 joints
Links:
- added link wall; collision box size=0.04 1.20 1.20; visual box size=0.04 1.20 1.20
Joints:
- added joint world_to_wall_joint: type fixed, parent world, child wall, origin xyz=0.8 0 0.75 rpy=0 0 0

Commit message: UPDATE: add new box obstacle for ur5

File: description/ur5/urdf/ur5.urdf (robot description, URDF)
Before this commit: robot ur5, 13 links, 12 joints
Links:
- added link box; collision box size=0.25 0.25 0.25; visual box size=0.25 0.25 0.25
- link wall: geometry collision box size=0.01 1.20 1.20; visual box size=0.04 1.20 1.20
Joints:
- added joint world_to_box_joint: type fixed, parent world, child box, origin xyz=0.7 0 0.5 rpy=0 0 0

Commit message: Update box location in ur5

File: description/ur5/urdf/ur5.urdf (robot description, URDF)
Before this commit: robot ur5, 14 links, 13 joints
Joints:
- joint world_to_box_joint: origin xyz=0.7 0 0.5 rpy=0 0 0 -> xyz=0.4 0.2 0.85 rpy=0 0 0

Commit message: Update wall params in ur5 urdf

File: description/ur5/urdf/ur5.urdf (robot description, URDF)
Before this commit: robot ur5, 14 links, 13 joints
Links:
- link wall: geometry collision box size=0.001 1.60 1.60; visual box size=0.001 1.60 1.60
Joints:
- joint world_to_wall_joint: origin xyz=0.8 0 0.75 rpy=0 0 0 -> xyz=0.8 0 0.8 rpy=0 0 0
