Commit message: MESH: rviz UR5 meshes in this repo, coloured like the MuJoCo model
The URDFs drew the UR5 from ocs2_robotic_assets' .dae meshes, whose embedded
colours did not show in rviz on Jazzy: the arm fell back to the URDF's uniform
LightGrey. Each UR link now has one visual per coloured part - STL copies of
this repo's MuJoCo OBJ parts, with the MuJoCo material colour - and the
collisions use this repo's STLs, so nothing here depends on
ocs2_robotic_assets any more.

Co-Authored-By: Claude Opus 5.5 <noreply@anthropic.com>

File: description/dual_ur5/urdf/dual_ur5.urdf (robot description, URDF)
Before this commit: robot dual_ur5, 38 links, 37 joints
Links:
- link ur_arm1_base_link_inertia: geometry collision cylinder length=0.025 radius=0.08; visual mesh filename=package://dynamics_mpc_controller/description/common/ur5_rv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
- link ur_arm1_forearm_link: geometry collision cylinder length=0.0885 radius=0.06; collision cylinder length=0.11 radius=0.038
- link ur_arm1_shoulder_link: geometry collision cylinder length=0.135 radius=0.06; visual mesh filename=package://dynamics_mpc_controller/description/common/ur5_rv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
- link ur_arm1_upper_arm_link: geometry collision cylinder length=0.1405 radius=0.06; collision cylinder length=0.143 radius=0.06
- link ur_arm1_wrist_1_link: geometry collision cylinder length=0.115 radius=0.038; visual mesh filename=package://dynamics_mpc_controller/description/common/ur5_rv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
- link ur_arm1_wrist_2_link: geometry collision cylinder length=0.105 radius=0.037; visual mesh filename=package://dynamics_mpc_controller/description/common/ur5_rv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
- link ur_arm1_wrist_3_link: geometry collision cylinder length=0.0065 radius=0.033; collision cylinder length=0.028 radius=0.04
- link ur_arm2_base_link_inertia: geometry collision cylinder length=0.025 radius=0.08; visual mesh filename=package://dynamics_mpc_controller/description/common/ur5_rv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
- link ur_arm2_forearm_link: geometry collision cylinder length=0.0885 radius=0.06; collision cylinder length=0.11 radius=0.038
- link ur_arm2_shoulder_link: geometry collision cylinder length=0.135 radius=0.06; visual mesh filename=package://dynamics_mpc_controller/description/common/ur5_rv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
- link ur_arm2_upper_arm_link: geometry collision cylinder length=0.1405 radius=0.06; collision cylinder length=0.143 radius=0.06
- link ur_arm2_wrist_1_link: geometry collision cylinder length=0.115 radius=0.038; visual mesh filename=package://dynamics_mpc_controller/description/common/ur5_rv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
- link ur_arm2_wrist_2_link: geometry collision cylinder length=0.105 radius=0.037; visual mesh filename=package://dynamics_mpc_controller/description/common/ur5_rv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
- link ur_arm2_wrist_3_link: geometry collision cylinder length=0.0065 radius=0.033; collision cylinder length=0.028 radius=0.04

File: description/ur5/urdf/ur5.urdf (robot description, URDF)
Before this commit: robot ur5, 14 links, 13 joints
Links:
- link ur_arm_base_link_inertia: geometry collision cylinder length=0.025 radius=0.08; visual mesh filename=package://dynamics_mpc_controller/description/common/ur5_rv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
- link ur_arm_forearm_link: geometry collision cylinder length=0.0885 radius=0.06; collision cylinder length=0.11 radius=0.038
- link ur_arm_shoulder_link: geometry collision cylinder length=0.135 radius=0.06; visual mesh filename=package://dynamics_mpc_controller/description/common/ur5_rv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
- link ur_arm_upper_arm_link: geometry collision cylinder length=0.1405 radius=0.06; collision cylinder length=0.143 radius=0.06
- link ur_arm_wrist_1_link: geometry collision cylinder length=0.115 radius=0.038; visual mesh filename=package://dynamics_mpc_controller/description/common/ur5_rv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
- link ur_arm_wrist_2_link: geometry collision cylinder length=0.105 radius=0.037; visual mesh filename=package://dynamics_mpc_controller/description/common/ur5_rv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
- link ur_arm_wrist_3_link: geometry collision cylinder length=0.0065 radius=0.033; collision cylinder length=0.028 radius=0.04
